File: hardware/racer-sensors/sensors.kicad_pcb (KiCad board)
At the start: 4 copper layers, 15.2 x 9 mm, 14 parts, among them J1 Conn_02x03_SMT, U1 OPT4060DTSR, U2 HAL1501SU-A

Commit message: hardware: sensors.kicad_pcb: Fix values of R1 and R2
Parts:
- R1, R2: value R -> 470
Changed lines of the file:
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@@
 			)
 		)
-		(property "Value" "R"
+		(property "Value" "470"
 			(at 0 1.43 180)
 			(layer "F.Fab")
@@
 			)
 		)
-		(property "Value" "R"
+		(property "Value" "470"
 			(at 0 1.43 180)
 			(layer "F.Fab")
