File: hardware/thumbtroller/controller.kicad_sch (KiCad schematic)
At the start: 61 parts, among them J11 UART, J12 JST 2.0 BATT, J9 Chip Enable, P1 USB_C_Plug_USB2.0, U1 THB001P, U5 ESP32-H2-MINI-1, U6 AP2204, U7 MCP73833

Commit message: Schematic readability update
Updated Schematics to hierarchical, Schematic size to A4.
Parts:
- removed C1, C10, C2, C3, C4: 1uF 25V, Capacitor_SMD:C_0603_1608Metric, symbol Device:C
- removed C11, C12, C13: 0.1uF, Capacitor_SMD:C_0603_1608Metric, symbol Device:C
- removed C14: 2.2uF, Capacitor_SMD:C_0603_1608Metric, symbol SAMC21_breakout-rescue:C
- removed C15: 10uF, Capacitor_SMD:C_0603_1608Metric, symbol SAMC21_breakout-rescue:C
- removed C16: 10uF, Capacitor_SMD:C_0603_1608Metric, symbol Device:C
- removed C17: 22uF, Capacitor_SMD:C_0603_1608Metric, symbol Device:C
- removed C9: 47uF, Capacitor_SMD:C_0603_1608Metric, symbol Device:C
- removed D1, D2, D3, D8, D9: LED, Capacitor_SMD:C_0603_1608Metric, symbol SAMC21_breakout-rescue:LED-RESCUE-SAMC21_breakout
- removed D5: TPD1E10B06DPYR, Diode_SMD:D_SOD-523, symbol custom_IC:TPD1E10B06DPYR
- removed D6: PWLED, Diode_SMD:D_0603_1608Metric, symbol Device:LED
- removed J11: UART, Connector_PinHeader_2.54mm:PinHeader_1x04_P2.54mm_Vertical, symbol Connector:Conn_01x04_Male
- removed J12: JST 2.0 BATT, Connector_JST:JST_PH_B2B-PH-K_1x02_P2.00mm_Vertical, symbol Connector_Generic:Conn_01x02
- removed J9: Chip Enable, Connector_PinHeader_2.54mm:PinHeader_1x02_P2.54mm_Vertical, symbol Connector:Conn_01x02_Male
- removed P1: USB_C_Plug_USB2.0, kicad_reformed_custom_IC:GCT_USB4105-GF-A, symbol Connector:USB_C_Plug_USB2.0
- removed R1, R12, R13, R25: 200, Resistor_SMD:R_0603_1608Metric, symbol SAMC21_breakout-rescue:R
- removed R10, R11, R2, R4, R6, R8, R9: 10k, Resistor_SMD:R_0603_1608Metric, symbol Device:R
- removed R14, R3, R5, R7: 100k, Resistor_SMD:R_0603_1608Metric, symbol Device:R
- removed R16: 1M, Resistor_SMD:R_0603_1608Metric, symbol Device:R
- removed R17, R18: 5k1, Resistor_SMD:R_0603_1608Metric, symbol Device:R
- removed R20, R21: 470, Resistor_SMD:R_0603_1608Metric, symbol Device:R
- removed R22, R23: 1.43K, Resistor_SMD:R_0603_1608Metric, symbol Device:R
- removed R24: 75K, Resistor_SMD:R_0603_1608Metric, symbol Device:R
- removed S1: JS102011SAQN, kicad_reformed_custom_IC:SW_JS102011SAQN, symbol custom_IC:JS102011SAQN
- removed S2, S3, S4, S5, S6: TL4100AF240QG_, kicad_reformed_custom_IC:SW_PTS810_SJM_250_SMTR_LFS, symbol custom_IC:TL4100AF240QG_
- removed TH1: TH 10k, Resistor_SMD:R_0603_1608Metric, symbol Device:Thermistor
- removed TP1: 0_IN1, TestPoint:TestPoint_Pad_1.0x1.0mm, symbol Connector:TestPoint
- removed TP2: 0_IN2, TestPoint:TestPoint_Pad_1.0x1.0mm, symbol Connector:TestPoint
- removed TP3: TP, TestPoint:TestPoint_Pad_D1.0mm, symbol Connector:TestPoint
- removed U1: THB001P, kicad_reformed_custom_IC:CNK_THB001P, symbol custom_IC:THB001P
- removed U5: ESP32-H2-MINI-1, kicad_reformed_custom_IC:MODULE_ESP32-H2-MINI-1-H2, symbol custom_IC:ESP32-H2-MINI-1
- removed U6: AP2204, kicad_reformed_custom_IC:AP2204, symbol SAMC21_breakout-rescue:AP2204
- removed U7: MCP73833, kicad_reformed_custom_IC:SON50P300X300X100-11N, symbol custom_IC:MCP73833
Connections:
- no-connect marks 14 -> 0
Other:
- added sheet Microcontroller (MCU.kicad_sch)
- added sheet Power (PWR.kicad_sch)
- note added: "Controller"
- note added: "Micro Racer Car"
- note removed: "BATT measurement"
- note removed: "Boot"
- note removed: "Charger"
- note removed: "Charging via USB C"
- note removed: "Connection Status"
- note removed: "GPIO8 LOG Boot Option"
- note removed: "GPIO9 needs to be HIGH on boot unless being programmed"
- note removed: "GREEN LED"
- note removed: "MCU Power"
- note removed: "Misc"
- note removed: "Power Status"
- note removed: "RC delay for chip EN"
- note removed: "RED LED"
- note removed: "Signals to MCU indicating state of charge"
- note removed: "USB C Power Only"
- note removed: "USB4105-GF-A"
- note removed: "replace with 10K?"
