File: hardware/racer/racer.kicad_pcb (KiCad board)
At the start: 4 copper layers, 36 x 50.2 mm, 83 parts, among them J1 motor0, J11 UART, J12 JST 2.0 BATT, J2 motor1, J3 motor0, J4 motor1, J5 motor0, J6 motor1, J7 motor0, J8 motor1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

Commit message: Update PCB from schematic
fixes pad <-> pin assignment

Signed-off-by: Andreas Heinrich <andreas.heinrich@rwth-aachen.de>
Connections:
- P1 pad S1: Net-(P1-SHIELD) -> Net-(P1-SHIELD-PadS1)
- P1 pad S2: (no net) -> Net-(P1-SHIELD-PadS1)
- R16 pad 1: Net-(P1-SHIELD) -> Net-(P1-SHIELD-PadS1)
Routing:
- net Net-(P1-SHIELD-PadS1): track 0.00 -> 4.95 mm
- net Net-(P1-SHIELD): track 4.95 -> 0.00 mm
Changed lines of the file:
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@@
 	(net 25 "Net-(U5-IO25)")
 	(net 26 "Net-(U5-IO22)")
-	(net 27 "Net-(P1-SHIELD)")
-	(net 28 "Net-(P1-VCONN)")
-	(net 29 "Net-(P1-CC)")
+	(net 27 "Net-(P1-SHIELD-PadS1)")
+	(net 28 "Net-(P1-CC2)")
+	(net 29 "Net-(P1-CC1)")
 	(net 30 "/STAT1")
 	(net 31 "/STAT2")
@@
 			(layers "F.Cu" "F.Paste" "F.Mask")
 			(roundrect_rratio 0.25)
-			(net 28 "Net-(P1-VCONN)")
+			(net 28 "Net-(P1-CC2)")
 			(pintype "passive")
 		)
@@
 			)
 		)
-		(property "Description" ""
+		(property "Description" "USB Power-Only 6P Type-C Receptacle connector"
 			(at 0 0 0)
 			(unlocked yes)
@@
 			)
 		)
-		(property ki_fp_filters "USB*C*Plug*")
+		(property ki_fp_filters "USB*C*Receptacle*")
 		(sheetname "Root")
 		(sheetfile "racer.kicad_sch")
@@
 			(size 0.7 2)
 			(layers "F.Cu" "F.Paste" "F.Mask")
-			(net 29 "Net-(P1-CC)")
-			(pinfunction "CC")
+			(net 29 "Net-(P1-CC1)")
+			(pinfunction "CC1")
 			(pintype "bidirectional")
 			(solder_mask_margin 0.102)
@@
 			(size 0.7 2)
 			(layers "F.Cu" "F.Paste" "F.Mask")
-			(net 28 "Net-(P1-VCONN)")
-			(pinfunction "VCONN")
+			(net 28 "Net-(P1-CC2)")
+			(pinfunction "CC2")
 			(pintype "bidirectional")
 			(solder_mask_margin 0.102)
@@
 			(layers "*.Cu" "*.Mask")
 			(remove_unused_layers no)
-			(net 27 "Net-(P1-SHIELD)")
+			(net 27 "Net-(P1-SHIELD-PadS1)")
 			(pinfunction "SHIELD")
 			(pintype "passive")
@@
 			(layers "*.Cu" "*.Mask")
 			(remove_unused_layers no)
+			(net 27 "Net-(P1-SHIELD-PadS1)")
+			(pinfunction "SHIELD")
+			(pintype "passive")
 			(solder_mask_margin 0.102)
 		)
@@
 			(layers "F.Cu" "F.Paste" "F.Mask")
 			(roundrect_rratio 0.25)
-			(net 29 "Net-(P1-CC)")
+			(net 29 "Net-(P1-CC1)")
 			(pintype "passive")
 		)
@@
 			(layers "F.Cu" "F.Paste" "F.Mask")
 			(roundrect_rratio 0.25)
-			(net 27 "Net-(P1-SHIELD)")
+			(net 27 "Net-(P1-SHIELD-PadS1)")
 			(pintype "passive")
 		)
