File: hardware/racer/racer.kicad_pcb (KiCad board)
At the start: 4 copper layers, 36 x 50.2 mm, 83 parts, among them J1 motor0, J11 UART, J12 JST 2.0 BATT, J2 motor1, J3 motor0, J4 motor1, J5 motor0, J6 motor1, J7 motor0, J8 motor1, J9 Conn_02x03_SMT, P1 USB_C_Plug_USB2.0, U1 A3908, U2 A3908, U3 A3908, U4 A3908, U5 ESP32-H2-MINI-1, U6 AP2204, U7 MCP73833

Commit message: hardware: racer.kicad_pcb: Fix wrong value of R22
Parts:
- R22: value 1.43K -> 5K
Changed lines of the file:
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@@
 			)
 		)
-		(property "Value" "1.43K"
+		(property "Value" "5K"
 			(at 0 1.43 90)
 			(layer "F.Fab")

Commit message: hardware version 1.0
Parts:
- removed D1, D2, D3, D4: LED, Capacitor_SMD:C_0603_1608Metric
- removed D6: PWLED, Diode_SMD:D_0603_1608Metric
- removed J11: UART, Connector_PinHeader_2.54mm:PinHeader_1x04_P2.54mm_Vertical
- removed R10, R30, R7: 10k, Resistor_SMD:R_0603_1608Metric
- removed R12, R13, R14, R15, R25: 200, Resistor_SMD:R_0603_1608Metric
- removed R8: 30k, Resistor_SMD:R_0603_1608Metric
- removed S3: TL4100AF240QG_, kicad_reformed_custom_IC:SW_PTS810_SJM_250_SMTR_LFS
- removed TP1, TP6: TP, TestPoint:TestPoint_Pad_D1.0mm
- added C18: 10uF, Capacitor_SMD:C_0603_1608Metric, F.Cu at (191.1, 100.6)
- added C19: 10uF, Capacitor_SMD:C_0603_1608Metric, F.Cu at (191.1, 99.0)
- added C20: 10uF, Capacitor_SMD:C_0603_1608Metric, F.Cu at (191.1, 105.5)
- added C21: 10uF, Capacitor_SMD:C_0603_1608Metric, F.Cu at (193.8, 95.7)
- added C22: 10uF, Capacitor_SMD:C_0603_1608Metric, F.Cu at (199.9, 95.5)
- added C23: 0.1uF, Capacitor_SMD:C_0603_1608Metric, F.Cu at (197.4, 131.9)
- added C24: 0.1uF, Capacitor_SMD:C_0603_1608Metric, F.Cu at (172.5, 132.0)
- added C25: 0.1uF, Capacitor_SMD:C_0603_1608Metric, F.Cu at (187.2, 117.4)
- added J10: Conn_02x03_SMT, Connector_PinHeader_1.27mm:PinHeader_2x03_P1.27mm_Vertical_SMD, F.Cu at (184.8, 123.8)
- added L1: 1uH, custom_IC:RES_CIGT252010, F.Cu at (187.3, 103.0)
- added LED1: IN-PI15TAT5R5G5B, custom_IC:IN-PI15_INL, F.Cu at (172.5, 88.8)
- added LED2: IN-PI15TAT5R5G5B, custom_IC:IN-PI15_INL, F.Cu at (197.3, 88.8)
- added LED3: IN-PI15TAT5R5G5B, custom_IC:IN-PI15_INL, F.Cu at (197.3, 135.0)
- added LED4: IN-PI15TAT5R5G5B, custom_IC:IN-PI15_INL, F.Cu at (172.5, 135.0)
- added LED5: IN-PI15TAT5R5G5B, custom_IC:IN-PI15_INL, F.Cu at (185.1, 118.6)
- added Q1: BSS138, Package_TO_SOT_SMD:SOT-23, F.Cu at (180.3, 100.5)
- added TP2: TestPoint, TestPoint:TestPoint_Pad_1.5x1.5mm, B.Cu at (178.9, 119.0)
- added U9: TPS631000DRLR, custom_IC:TPS631000DRLR_TEX, F.Cu at (191.1, 103.0)
- C10: value 1uF 25V -> 1uF
- C14: value 2.2uF -> 0.1uF
- C15: value 10uF -> 0.1uF
- C17: value 22uF -> 47uF
- D5: value TPD1E10B06DPYR -> TPD1E10B06
- D8: value LED -> LED_GREEN
- D9: value LED -> LED_RED
- G***: moved to B.Cu
- P1: footprint kicad_reformed_custom_IC:CUI_UJC-VP-3-SMT-TR -> kicad_reformed_custom_IC:GCT_USB4105-GF-A
- R1, R11, R9: value 10k -> 10K
- R17, R18: value 5k1 -> 5K1
- R2: value 30k -> 806
- R20, R21: value 200 -> 330
- R22: value 5K -> 5K1
- R26, R27, R28, R29: value 100k -> 10K
- R3: value 10k -> 91
- R4, R6: value 30k -> 10K
- R5: value 10k -> 470
- REF**: moved to F.Cu
- S2: value TL4100AF240QG_ -> SWITCH_0SMTRLFS; footprint kicad_reformed_custom_IC:SW_PTS810_SJM_250_SMTR_LFS -> kicad_reformed_custom_IC:SWITCH_0SMTRLFS
- TH1: value TH 10k -> TH 10K
- U6: value AP2204 -> AP2205
- moved G*** 40.4 mm to (199.8, 133.3), turned to 180 degrees
- moved R6 30.8 mm to (194.3, 105.5), turned to 180 degrees
- moved R5 29.6 mm to (176.7, 101.0), turned to 180 degrees
- moved REF** 28.6 mm to (169.8, 125.3), turned to 90 degrees
- moved C14 28.4 mm to (174.0, 91.5), turned to -90 degrees
- moved R20 25.5 mm to (174.5, 125.7), turned to 0 degrees
- moved D8 23.0 mm to (177.6, 125.7), turned to 180 degrees
- moved R21 21.3 mm to (174.5, 122.8), turned to 0 degrees
- moved R16 20.7 mm to (200.4, 130.0), turned to -90 degrees
- moved R2 20.0 mm to (193.9, 100.0), turned to -90 degrees
- moved D9 18.4 mm to (177.6, 122.8), turned to 180 degrees
- moved R4 17.7 mm to (176.7, 99.4)
- moved P1 15.3 mm to (200.1, 122.6), turned to 90 degrees
- moved R1 13.4 mm to (182.8, 100.9)
- moved R3 9.99 mm to (193.9, 103.1)
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Connections:
- net /STAT1 renamed /STAT1_CHARGING
- net /STAT2 renamed /STAT2_DONE
- C14 pad 1: RAW -> +5V
- C15 pad 1: +3V3 -> +5V
- C16 pad 1: +5V -> +5VD
- D5 pad 1: +5V -> +5VD
- P1 pad A9: +5V -> +5VD
- R1 pad 1: Net-(U1-VREF) -> Net-(Q1-S)
- R1 pad 2: Net-(U1-VSET) -> +3V3
- R2 pad 1: Net-(U1-VSET) -> +5V
- R2 pad 2: GND -> Net-(U9-FB)
- R20 pad 1: +5V -> +5VD
- R21 pad 1: +5V -> +5VD
- R3 pad 1: Net-(U2-VREF) -> Net-(U9-FB)
- R3 pad 2: Net-(U2-VSET) -> GND
- R4 pad 1: Net-(U2-VSET) -> Net-(Q1-D)
- R4 pad 2: GND -> +5V
- R5 pad 1: Net-(U3-VREF) -> Net-(Q1-D)
- R5 pad 2: Net-(U3-VSET) -> Net-(LED1-DIN)
- R6 pad 1: Net-(U3-VSET) -> GND
- R6 pad 2: GND -> Net-(U9-MODE)
- S2 pad 1: Net-(U5-IO9) -> GND
- S2 pad 2: GND -> Net-(U5-IO9)
- U1 pad 5: Net-(U1-VSET) -> Net-(U1-VREF)
- U2 pad 5: Net-(U2-VSET) -> Net-(U2-VREF)
- U3 pad 5: Net-(U3-VSET) -> Net-(U3-VREF)
- U4 pad 5: Net-(U4-VSET) -> Net-(U4-VREF)
- U5 pad 16: unconnected-(U5-IO12-Pad16) -> /IO12
- U5 pad 21: Net-(U5-IO11) -> /IO11
- U5 pad 24: Net-(U5-IO22) -> /IO22
- U5 pad 25: Net-(U5-IO25) -> Net-(Q1-S)
- U5 pad 26: Net-(U5-IO26) -> /USB_D-
- U5 pad 27: Net-(U5-IO27) -> /USB_D+
- U5 pad 30: /U0RXD -> unconnected-(U5-RXD0-Pad30)
- U5 pad 31: /U0TXD -> unconnected-(U5-TXD0-Pad31)
- U5 pad 5: /ADC_BATT -> LIPO+
- U5 pad 6: Net-(U5-IO3) -> /OPT_INT
- U6 pad 1: RAW -> +5V
- U6 pad 3: RAW -> +5V
- U7 pad 1: +5V -> +5VD
- U7 pad 2: +5V -> +5VD
Routing:
- net Net-(LED2-DOUT): track 0.00 -> 51.5 mm, vias 0 -> 2
- net Net-(U5-IO26): track 44.2 -> 0.00 mm, vias 2 -> 0
- net +5VD: track 0.00 -> 39.1 mm
- net Net-(U5-IO27): track 35.3 -> 0.00 mm, vias 2 -> 0
- net /USB_D+: track 0.00 -> 32.8 mm, vias 0 -> 2
- net /ADC_BATT: track 31.8 -> 0.00 mm, vias 2 -> 0
- net /USB_D-: track 0.00 -> 31.7 mm, vias 0 -> 2
- net Net-(LED4-DOUT): track 0.00 -> 31.5 mm, vias 0 -> 3
- net /IO22: track 0.00 -> 25.5 mm, vias 0 -> 2
- net /OPT_INT: track 0.00 -> 25.2 mm, vias 0 -> 2
- net Net-(U5-IO25): track 25.2 -> 0.00 mm, vias 2 -> 0
- net Net-(LED1-DOUT): track 0.00 -> 25.0 mm, vias 0 -> 2
- net Net-(LED3-DOUT): track 0.00 -> 24.8 mm, vias 0 -> 2
- net Net-(U5-IO22): track 24.7 -> 0.00 mm, vias 2 -> 0
- net /IO11: track 0.00 -> 20.9 mm, vias 0 -> 2
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- added copper zone on F.Cu, net +3V3
- added copper zone on F.Cu, net +5V
- added copper zone on In2.Cu, net +5V
- added copper zone on F.Cu, net Net-(U9-LX1)
- added copper zone on F.Cu, net Net-(U9-LX2)
- added copper zone on F.Cu, net RAW
Other:
- board text added: "Racer v1.0"
- board text added: "StuckAtPrototype"
- board text removed: "3v3"
- board text removed: "GND"
- board text removed: "REF"
- board text removed: "RXD"
- board text removed: "Racer v0.2"
- board text removed: "StuckAtPrototype DMsensors"
- board text removed: "TXD"
