File: hardware/racer/racer.kicad_sch (KiCad schematic)
At the start: 79 parts, among them J1 motor0, J11 UART, J12 JST 2.0 BATT, J2 motor1, J3 motor0, J4 motor1, J5 motor0, J6 motor1, J7 motor0, J8 motor1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

Commit message: Add part numbers to schematic
* Add property `MFR Part #`
* Add property `LCSC`

Signed-off-by: Andreas Heinrich <andreas.heinrich@rwth-aachen.de>
Parts:
- C1, C15, C16, C2, C5, C6: LCSC (none) -> C90053; MFR Part # (none) -> GRM188R61A106ME69D
- C10: LCSC (none) -> C14664; MFR Part # (none) -> CC0603KRX5R8BB105
- C11, C12, C13, C3, C4, C7, C8: LCSC (none) -> C108079; MFR Part # (none) -> CC0603KRX7R7BB104
- C14: LCSC (none) -> C23630; MFR Part # (none) -> CL10A225KO8NNNC
- C17: LCSC (none) -> C426040; MFR Part # (none) -> GRM188R60J226MEA0J
- C9: LCSC (none) -> C576468; MFR Part # (none) -> GRM188C80E476ME05D
- D1, D2, D6, D8, D9: LCSC (none) -> C3030991; MFR Part # (none) -> 150060RS75000
- D3, D4: LCSC (none) -> C7207730; MFR Part # (none) -> IN-S63AT5UW
- D5: LCSC (none) -> C3712135; MFR Part # (none) -> TPD1E10B06DYAR
- J11: LCSC (none) -> C29779969; MFR Part # (none) -> PZ2.54-1x4-11.2
- J12: LCSC (none) -> C20504437; MFR Part # (none) -> B2B-PH-K-S
- J9: LCSC (none) -> C5646308; MFR Part # (none) -> GRPB032VWQS-RC
- P1: LCSC (none) -> C5126695; MFR Part # (none) -> UJC-VP-3-SMT-TR
- R1, R10, R11, R3, R30, R5, R7, R9: LCSC (none) -> C384294; MFR Part # (none) -> WR06X103 JTL
- R12, R13, R14, R15, R20, R21, R25: LCSC (none) -> C2846665; MFR Part # (none) -> ESR03EZPF2000
- R16: LCSC (none) -> C237111; MFR Part # (none) -> RMCF0603FT1M00
- R17, R18: LCSC (none) -> C5126695; MFR Part # (none) -> RMCF0603JT5R10
- R2, R4, R6, R8: LCSC (none) -> C2085991; MFR Part # (none) -> ERA-3AED303V
- R22: LCSC (none) -> C2479774; MFR Part # (none) -> RMCF0603JT5R10
- R23: LCSC (none) -> C861730; MFR Part # (none) -> RT0603BRE071K43L
- R24: LCSC (none) -> C413688; MFR Part # (none) -> ERJ-PB3B7502V
- R26, R27, R28, R29: LCSC (none) -> C132374; MFR Part # (none) -> WR06X1003FTL
- S1: LCSC (none) -> C221660; MFR Part # (none) -> JS102011SAQN
- S2, S3: LCSC (none) -> C116501; MFR Part # (none) -> PTS810SJM250SMTRLFS
- TH1: LCSC (none) -> C531304; MFR Part # (none) -> NTCG163JF103HT1
- U1, U2, U3, U4: LCSC (none) -> C459250; MFR Part # (none) -> A3908EEETR-T
- U5: LCSC (none) -> C18203134; MFR Part # (none) -> ESP32-H2-MINI-1-N4
- U6: LCSC (none) -> C3750488; MFR Part # (none) -> AP2205-33W5-7
- U7: LCSC (none) -> C340160; MFR Part # (none) -> MCP73833T-AMI/MF

Commit message: Rename field to MPN
Signed-off-by: Andreas Heinrich <andreas.heinrich@rwth-aachen.de>
Parts:
- C1, C15, C16, C2, C5, C6: MFR Part # GRM188R61A106ME69D -> (none); MPN (none) -> GRM188R61A106ME69D
- C10: MFR Part # CC0603KRX5R8BB105 -> (none); MPN (none) -> CC0603KRX5R8BB105
- C11, C12, C13, C3, C4, C7, C8: MFR Part # CC0603KRX7R7BB104 -> (none); MPN (none) -> CC0603KRX7R7BB104
- C14: MFR Part # CL10A225KO8NNNC -> (none); MPN (none) -> CL10A225KO8NNNC
- C17: MFR Part # GRM188R60J226MEA0J -> (none); MPN (none) -> GRM188R60J226MEA0J
- C9: MFR Part # GRM188C80E476ME05D -> (none); MPN (none) -> GRM188C80E476ME05D
- D1, D2, D6, D8, D9: MFR Part # 150060RS75000 -> (none); MPN (none) -> 150060RS75000
- D3, D4: MFR Part # IN-S63AT5UW -> (none); MPN (none) -> IN-S63AT5UW
- D5: MFR Part # TPD1E10B06DYAR -> (none); MPN (none) -> TPD1E10B06DYAR
- J11: MFR Part # PZ2.54-1x4-11.2 -> (none); MPN (none) -> PZ2.54-1x4-11.2
- J12: MFR Part # B2B-PH-K-S -> (none); MPN (none) -> B2B-PH-K-S
- J9: MFR Part # GRPB032VWQS-RC -> (none); MPN (none) -> GRPB032VWQS-RC
- P1: MFR Part # UJC-VP-3-SMT-TR -> (none); MPN (none) -> UJC-VP-3-SMT-TR
- R1, R10, R11, R3, R30, R5, R7, R9: MFR Part # WR06X103 JTL -> (none); MPN (none) -> WR06X103 JTL
- R12, R13, R14, R15, R20, R21, R25: MFR Part # ESR03EZPF2000 -> (none); MPN (none) -> ESR03EZPF2000
- R16: MFR Part # RMCF0603FT1M00 -> (none); MPN (none) -> RMCF0603FT1M00
- R17, R18, R22: MFR Part # RMCF0603JT5R10 -> (none); MPN (none) -> RMCF0603JT5R10
- R2, R4, R6, R8: MFR Part # ERA-3AED303V -> (none); MPN (none) -> ERA-3AED303V
- R23: MFR Part # RT0603BRE071K43L -> (none); MPN (none) -> RT0603BRE071K43L
- R24: MFR Part # ERJ-PB3B7502V -> (none); MPN (none) -> ERJ-PB3B7502V
- R26, R27, R28, R29: MFR Part # WR06X1003FTL -> (none); MPN (none) -> WR06X1003FTL
- S1: MFR Part # JS102011SAQN -> (none); MPN (none) -> JS102011SAQN
- S2, S3: MFR Part # PTS810SJM250SMTRLFS -> (none); MPN (none) -> PTS810SJM250SMTRLFS
- TH1: MFR Part # NTCG163JF103HT1 -> (none); MPN (none) -> NTCG163JF103HT1
- U1, U2, U3, U4: MFR Part # A3908EEETR-T -> (none); MPN (none) -> A3908EEETR-T
- U5: MFR Part # ESP32-H2-MINI-1-N4 -> (none); MPN (none) -> ESP32-H2-MINI-1-N4
- U6: MFR Part # AP2205-33W5-7 -> (none); MPN (none) -> AP2205-33W5-7
- U7: MFR Part # MCP73833T-AMI/MF -> (none); MPN (none) -> MCP73833T-AMI/MF
