File: hardware/racer/racer.kicad_sch (KiCad schematic)
At the start: 79 parts, among them J1 motor0, J11 UART, J12 JST 2.0 BATT, J2 motor1, J3 motor0, J4 motor1, J5 motor0, J6 motor1, J7 motor0, J8 motor1, J9 Conn_02x03_SMT, P1 USB_C_Plug_USB2.0, U1 A3908, U2 A3908, U3 A3908, U4 A3908, U5 ESP32-H2-MINI-1, U6 AP2204, U7 MCP73833

Commit message: hardware version 1.0
Parts:
- removed C1, C15, C2, C5, C6: 10uF, Capacitor_SMD:C_0603_1608Metric, symbol SAMC21_breakout-rescue:C
- removed C14: 2.2uF, Capacitor_SMD:C_0603_1608Metric, symbol SAMC21_breakout-rescue:C
- removed C3, C4, C7, C8: 0.1uF, Capacitor_SMD:C_0603_1608Metric, symbol SAMC21_breakout-rescue:C
- removed D1, D2, D3, D4: LED, Capacitor_SMD:C_0603_1608Metric, symbol SAMC21_breakout-rescue:LED-RESCUE-SAMC21_breakout
- removed D6: PWLED, Diode_SMD:D_0603_1608Metric, symbol Device:LED
- removed J1, J3, J5, J7: motor0, TestPoint:TestPoint_Pad_2.0x2.0mm, symbol SAMC21_breakout-rescue:Conn_01x01_Female-Connector
- removed J11: UART, Connector_PinHeader_2.54mm:PinHeader_1x04_P2.54mm_Vertical, symbol Connector:Conn_01x04_Male
- removed J2, J4, J6, J8: motor1, TestPoint:TestPoint_Pad_2.0x2.0mm, symbol SAMC21_breakout-rescue:Conn_01x01_Female-Connector
- removed R10, R30, R7: 10k, Resistor_SMD:R_0603_1608Metric, symbol Device:R
- removed R12, R13, R14, R15, R25: 200, Resistor_SMD:R_0603_1608Metric, symbol SAMC21_breakout-rescue:R
- removed R8: 30k, Resistor_SMD:R_0603_1608Metric, symbol Device:R
- removed S3: TL4100AF240QG_, kicad_reformed_custom_IC:SW_PTS810_SJM_250_SMTR_LFS, symbol custom_IC:TL4100AF240QG_
- removed TP1, TP6: TP, TestPoint:TestPoint_Pad_D1.0mm, symbol Connector:TestPoint
- removed U1, U2, U3, U4: A3908, kicad_reformed_custom_IC:A3908, symbol SAMC21_breakout-rescue:A3908-custom_IC
- added C14, C15, C23, C24, C25: 0.1uF, Capacitor_SMD:C_0603_1608Metric, symbol Device:C
- added C18, C19, C20: 10uF, Capacitor_SMD:C_0603_1608Metric, symbol Device:C
- added C21, C22: 10uF, Capacitor_SMD:C_0603_1608Metric, symbol SAMC21_breakout-rescue:C
- added J10: Conn_02x03_SMT, Connector_PinHeader_1.27mm:PinHeader_2x03_P1.27mm_Vertical_SMD, symbol Connector:Conn_01x06_Pin
- added L1: 1uH, custom_IC:RES_CIGT252010, symbol Device:L
- added LED1, LED2, LED3, LED4, LED5: IN-PI15TAT5R5G5B, custom_IC:IN-PI15_INL, symbol custom_IC:IN-PI15TAT5R5G5B
- added Q1: BSS138, Package_TO_SOT_SMD:SOT-23, symbol Transistor_FET:BSS138
- added TP2: TestPoint, TestPoint:TestPoint_Pad_1.5x1.5mm, symbol Connector:TestPoint
- added U9: TPS631000DRLR, custom_IC:TPS631000DRLR_TEX, symbol custom_IC:TPS631000DRLR
- C10: value 1uF 25V -> 1uF
- C17: value 22uF -> 47uF
- D5: value TPD1E10B06DPYR -> TPD1E10B06
- D8: value LED -> LED_GREEN
- D9: value LED -> LED_RED
- P1: footprint kicad_reformed_custom_IC:CUI_UJC-VP-3-SMT-TR -> kicad_reformed_custom_IC:GCT_USB4105-GF-A
- R1, R11, R9: value 10k -> 10K
- R17, R18: value 5k1 -> 5K1
- R2: value 30k -> 806
- R20, R21: value 200 -> 330
- R22: value 5K -> 5K1
- R26, R27, R28, R29: value 100k -> 10K
- R3: value 10k -> 91
- R4, R6: value 30k -> 10K
- R5: value 10k -> 470
- S2: value TL4100AF240QG_ -> SWITCH_0SMTRLFS; footprint kicad_reformed_custom_IC:SW_PTS810_SJM_250_SMTR_LFS -> kicad_reformed_custom_IC:SWITCH_0SMTRLFS
- TH1: value TH 10k -> TH 10K
- U6: value AP2204 -> AP2205
Connections:
- net ADC_BATT is gone; now on net LIPO+: U5.5 (IO2)
- net +3V3: now also R1.2, C22.1, J10.2 (Pin_2), Q1.1 (G)
- net +5V: now also R2.1, R4.2, U6.1 (VIN), U6.3 (EN), C14.1, C15.1, C18.1, C19.1, C21.1, C23.1, C24.1, C25.1, LED1.2 (VDD), LED2.2 (VDD), LED3.2 (VDD), LED4.2 (VDD), LED5.2 (VDD), U9.1 (VOUT); no longer C16.1, D5.1, P1.A4 (VBUS), P1.A9 (VBUS), P1.B4 (VBUS), P1.B9 (VBUS), R20.1, R21.1, U7.1 (VDD), U7.2 (VDD)
- net CP_EN: now also TP2.1
- net GND: now also R3.2, R6.1, S2.1, C14.2, C15.2, C18.2, C19.2, C20.2, C21.2, C22.2, C23.2, C24.2, C25.2, J10.5 (Pin_5), LED1.4 (GND), LED2.4 (GND), LED3.4 (GND), LED4.4 (GND), LED5.4 (GND), U9.7 (GND); no longer R2.2, R4.2, R6.2, S2.2
- net OPT_INT: now also U5.6 (IO3)
- net RAW: now also C20.1, U9.4 (VIN), U9.5 (EN); no longer U6.1 (VIN), U6.3 (EN)
- net at R1.1: now also U5.25 (IO25), Q1.2 (S)
- net at R5.2: now also LED1.1 (DIN); no longer R6.1
- net IO12: now reaches U5.16 (IO12)
- net IO12: now also J10.3 (Pin_3)
- net IO11: now reaches U5.21 (IO11)
- net IO11: now also J10.4 (Pin_4)
- net at U5.23 (IO9): now also S2.2; no longer S2.1
- net IO22: now reaches U5.24 (IO22)
- net IO22: now also J10.6 (Pin_6)
- net USB_D-: now reaches U5.26 (IO26)
- net USB_D-: now also P1.A7 (D-)
- net USB_D+: now reaches U5.27 (IO27)
- net USB_D+: now also P1.A6 (D+)
- net at R3.1: now also R2.2, U9.8 (FB)
- net at R4.1: now also R5.1, Q1.3 (D); no longer R3.2
- net MOTOR_0_IN1 renamed Motor drivers/MOTOR_0_IN1
- net MOTOR_0_IN2 renamed Motor drivers/MOTOR_0_IN2
- net MOTOR_1_IN1 renamed Motor drivers/MOTOR_1_IN1
- net MOTOR_1_IN2 renamed Motor drivers/MOTOR_1_IN2
- net STAT1 renamed STAT1_CHARGING
- net STAT2 renamed STAT2_DONE
- net U0RXD: no longer names the net of U5.30 (RXD0)
- net U0TXD: no longer names the net of U5.31 (TXD0)
- new net: LED4.3 (DOUT), LED5.1 (DIN)
- new net: L1.2, U9.2 (LX2)
- new net: L1.1, U9.3 (LX1)
- new net: R6.2, U9.6 (MODE)
- new net: LED2.3 (DOUT), LED3.1 (DIN)
- new net: LED3.3 (DOUT), LED4.1 (DIN)
- new net: LED1.3 (DOUT), LED2.1 (DIN)
- new net +5VD: C16.1, D5.1, P1.A4 (VBUS), P1.A9 (VBUS), P1.B4 (VBUS), P1.B9 (VBUS), R20.1, R21.1, U7.1 (VDD), U7.2 (VDD)
- no-connect marks 13 -> 14
Other:
- added sheet Motor drivers (motor_drivers.kicad_sch)
- note added: "5V"
- note added: "CIGT252010EH1R0MNE"
- note added: "Charging"
- note added: "Done"
- note added: "Front Left"
- note added: "Front Right"
- note added: "Info"
- note added: "Lets the USB controller know we want to charge"
- note added: "Lipo voltage is between 2.7V and 4.2V"
- note added: "Place close to U7"
- note added: "Power"
- note added: "Rear Left"
- note added: "Rear Right"
- note added: "Transistor for logic level shift"
- note added: "Using LEDs for charge status"
- note removed: "BATT measurement voltage/2"
- note removed: "Front and Back Lights"
- note removed: "MOTOR 0A"
- note removed: "MOTOR 0B"
- note removed: "MOTOR 1A"
- note removed: "MOTOR 1B"
- note removed: "Motor Ctrl"
- note removed: "NOTE: If voltage regulation is not needed, install a 0 Ohm resistor on R1 (x4)"
- note removed: "Signals to MCU indicating state of charge"
- note removed: "USB C Power Only"
- note removed: "replace with 10K?"
- company: StuckAtPrototype -> StuckAtPrototype LLC
- title: Racer -> Micro Racer
- moved on the sheet: C10, C11, C12, C13, C16, C17, C9, D5, D8, D9, J12, J9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
